File: Driver_Boards/NORITAKE_ITRON_MN12832JC.brd (EAGLE design)
At the start: 114.3 x 38.1 mm, 59 parts, among them IC1 CD74HC123ME4, J3 AVR_SPI_PROG_3X2PTH, Q1 220mA/50V/3.5Ω, Q2 20A/100V/110mΩ, U1 LTC6906CS6TRPBF, U2 MAX628CSA+, U3 32U4, U4 SN74LVC1G32DCKR, Y1 16MHz

Commit message: Itron Driver ready for protos
Parts:
- added U$10, U$12: (no value), output:#_5VDC#0
- added U$15, U$7: (no value), output:#GND#0
- added U$16: (no value), output:#_RXI#0
- added U$18: (no value), output:#_TXO#0
- added U$2: (no value), blueshire:BLUESHIRE_COPPER#SVG1
- added U$3: (no value), blueshire:BLUESHIRE_SILK#SVG0
- added U$4: (no value), blueshire:BLUESHIRE_STOP#SVG2
- added U$5: (no value), output:OPEN_SOURCE_HARDWARE_DRIVER0
- added U$6: (no value), output:FOR_NORITAKE_ITRON_MN12832JC0
- added U$8: (no value), output:#_SCL#0
- added U$9: (no value), output:#_SDA#0
- J1, J2: device SparkFun-Connectors:1X04 -> SparkFun-Connectors:1X04_NO_SILK
- moved J1 25.4 mm to (2.54, 36.8), turned to 0 degrees
- moved J2 23.9 mm to (22.9, 36.8), turned to 180 degrees
- moved C8 4.75 mm to (22.9, 31.8), turned to 270 degrees
- moved Y1 3.42 mm to (26.7, 31.8), turned to 90 degrees
- moved C9 2.18 mm to (30.5, 31.8), turned to 90 degrees
- moved C13 1.63 mm to (31.8, 18.8), turned to 180 degrees
Routing:
- net 5V: track 90.9 -> 189.8 mm, vias 0 -> 8
- net V_USB: track 0.00 -> 45.5 mm, vias 0 -> 4
- net TXO: track 0.00 -> 22.4 mm, vias 0 -> 1
- net RXI: track 0.00 -> 21.0 mm, vias 0 -> 1
- net SDA: track 0.00 -> 13.4 mm
- net SCL: track 0.00 -> 12.7 mm
- net RESET: track 20.9 -> 32.2 mm, vias 0 -> 1
- net N$6: track 0.00 -> 5.73 mm
- net WATCHDOG: track 20.2 -> 22.9 mm, vias 0 -> 2
- net UCAP: track 4.53 -> 2.35 mm
- net N$16: track 13.7 -> 12.0 mm
- net N$15: track 13.3 -> 13.9 mm
Other:
- board text added: "NPOOLE2021"
- board text added: "v0.01"
