File: Driver_Boards/NORITAKE_ITRON_MN12832JC.sch (EAGLE design)
At the start: 59 parts, among them IC1 CD74HC123ME4, J3 AVR_SPI_PROG_3X2PTH, Q1 220mA/50V/3.5Ω, Q2 20A/100V/110mΩ, U1 LTC6906CS6TRPBF, U2 MAX628CSA+, U3 32U4, U4 SN74LVC1G32DCKR, Y1 16MHz

Commit message: Itron Driver ready for protos
Parts:
- J1, J2: device SparkFun-Connectors:CONN_04PTH -> SparkFun-Connectors:CONN_041X04_NO_SILK
Changed lines of the file:
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@@
 <part name="SUPPLY16" library="SparkFun-PowerSymbols" deviceset="5V" device=""/>
 <part name="GND31" library="SparkFun-PowerSymbols" deviceset="GND" device=""/>
-<part name="J1" library="SparkFun-Connectors" deviceset="CONN_04" device="PTH"/>
+<part name="J1" library="SparkFun-Connectors" deviceset="CONN_04" device="1X04_NO_SILK"/>
 <part name="J3" library="SparkFun-Connectors" deviceset="AVR_SPI_PROG_3X2" device="PTH"/>
 <part name="GND33" library="SparkFun-PowerSymbols" deviceset="GND" device=""/>
@@
 <part name="SUPPLY18" library="SparkFun-PowerSymbols" deviceset="5V" device=""/>
 <part name="GND34" library="SparkFun-PowerSymbols" deviceset="GND" device=""/>
-<part name="J2" library="SparkFun-Connectors" deviceset="CONN_04" device="PTH"/>
+<part name="J2" library="SparkFun-Connectors" deviceset="CONN_04" device="1X04_NO_SILK"/>
 <part name="SUPPLY19" library="SparkFun-PowerSymbols" deviceset="5V" device=""/>
 <part name="GND35" library="SparkFun-PowerSymbols" deviceset="GND" device=""/>
